File: ECG_KICAD_Files/ECG_Project_Josh/ECG_Project_Josh.kicad_pcb (KiCad board)
At the start: 2 copper layers, 35 parts, among them J1 Conn_01x02_Pin, J2 Conn_01x02_Pin, J3 Conn_01x03_Pin, U1 LF412ACN/NOPB, U2 AD623AN, U3 LF412ACN/NOPB

Commit message: PCB Complete DRM Passed
Parts:
- J1, J2: moved to B.Cu
- moved J3 180.2 mm to (83.5, 97.6), turned to 180 degrees
- moved J1 167.9 mm to (83.5, 102.5), turned to 180 degrees
- moved J2 165.0 mm to (83.5, 63.0), turned to 180 degrees
- moved U3 164.7 mm to (105.3, 76.3), turned to 180 degrees
- moved U2 162.7 mm to (100.7, 98.2)
- moved C10 150.9 mm to (86.5, 79.2), turned to 90 degrees
- moved R18 148.3 mm to (83.5, 68.7), turned to -90 degrees
- moved C1 147.0 mm to (92.0, 83.2), turned to -90 degrees
- moved R1 147.0 mm to (86.4, 102.5)
- moved R17 145.1 mm to (83.5, 79.5), turned to -90 degrees
- moved R4 145.0 mm to (86.4, 105.0)
- moved R19 144.6 mm to (91.3, 60.5), turned to 180 degrees
- moved R16 142.1 mm to (89.5, 64.2), turned to -90 degrees
- moved C2 141.7 mm to (97.0, 85.2), turned to -90 degrees
- moved U1 137.7 mm to (115.4, 96.5)
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Connections:
- J3 pad 2: Vcc -> Vee
- J3 pad 3: Vee -> Vcc
Routing:
- net Vcc: track 0.00 -> 141.8 mm
- net Vee: track 0.00 -> 92.8 mm
- net Net-(U1A-IN+): track 0.00 -> 28.9 mm
- net Net-(U2-Vs+): track 0.00 -> 28.7 mm
- net Net-(U3A-OUT): track 0.00 -> 24.9 mm
- net Net-(U3A-IN-): track 0.00 -> 24.2 mm
- net Net-(U1B-IN-): track 0.00 -> 22.9 mm
- net Net-(C6-Pad1): track 0.00 -> 22.7 mm
- net Net-(U3B-IN-): track 0.00 -> 21.5 mm
- net Net-(U2-Vs-): track 0.00 -> 20.0 mm
- net Net-(J2-Pin_2): track 0.00 -> 19.2 mm
- net Net-(U1B-IN+): track 0.00 -> 18.9 mm
- net Net-(U3B-OUT): track 0.00 -> 12.0 mm
- net Net-(C4-Pad1): track 0.00 -> 11.2 mm
- net Net-(R2-Pad2): track 0.00 -> 10.7 mm
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- added copper zone on B.Cu, net GND
Other:
- board outline added: 66.5 x 53 mm
